File: SX1255_HAT-hw.kicad_sch (KiCad schematic)
At the start: 26 parts, among them IC1 SX1255, J1 TX_SMA, J2 RX_SMA, J3 RPi Zero, Y1 32MHz

Commit message: pcb update
Parts:
- added H1, H2, H3, H4: MountingHole, MountingHole:MountingHole_2.7mm_M2.5_DIN965, symbol Mechanical:MountingHole
- added R4: 100R, Resistor_SMD:R_0603_1608Metric, symbol Device:R_Small
- added SYM1: Logo_Open_Hardware_Small, Symbol:OSHW-Logo2_7.3x6mm_SilkScreen, symbol Graphic:Logo_Open_Hardware_Small
- IC1: footprint QFN50P500X500X80-33N-D -> parts:QFN50P500X500X80-33N-D
- renumbered R4 to R5, R5 to R6, R6 to R7
Connections:
- net DIO2: now also R4.1; no longer IC1.23 (DIO2)
- new net: IC1.23 (DIO2), R4.2

Commit message: BOM and silkscreen updates
Parts:
- C1, C2, C3, C4: MPN C0603C103K5RAC7081 -> 80-C0603C103M4RECLR; PN C0603C103K5RAC7081 -> 80-C0603C103M4RECLR
- C10, C13, C5, C6, C7, C8, C9: MPN C0603C104M5RAC7411 -> 581-06035G104Z; PN C0603C104M5RAC7411 -> 581-06035G104Z
- C11: MPN (none) -> 77-VJ0603A330KXAPBC; PN (none) -> 77-VJ0603A330KXAPBC
- C12: MPN (none) -> 603-AC0603JRNP9BN270; PN (none) -> 603-AC0603JRNP9BN270
- H1, H2, H3, H4, J3, SYM1: MPN (none) -> -; PN (none) -> -
- L1: MPN (none) -> 815-AISC-0603-R082-J; PN (none) -> 815-AISC-0603-R082-J
- L2: MPN (none) -> 815-AISC-0603-R039-J; PN (none) -> 815-AISC-0603-R039-J
Changed lines of the file:
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@@
 			)
 		)
-		(property "PN" "C0603C104M5RAC7411"
+		(property "PN" "581-06035G104Z"
 			(at 114.3 107.95 0)
 			(effects
@@
 			)
 		)
-		(property "MPN" "C0603C104M5RAC7411"
+		(property "MPN" "581-06035G104Z"
 			(at 114.3 107.95 0)
 			(effects
@@
 			)
 		)
-		(property "PN" "C0603C103K5RAC7081"
+		(property "PN" "80-C0603C103M4RECLR"
 			(at 58.42 139.7 0)
 			(effects
@@
 			)
 		)
-		(property "MPN" "C0603C103K5RAC7081"
+		(property "MPN" "80-C0603C103M4RECLR"
 			(at 58.42 139.7 0)
 			(effects
@@
 			)
 		)
-		(property "PN" "C0603C104M5RAC7411"
+		(property "PN" "581-06035G104Z"
 			(at 170.18 76.2 0)
 			(effects
@@
 			)
 		)
-		(property "MPN" "C0603C104M5RAC7411"
+		(property "MPN" "581-06035G104Z"
 			(at 170.18 76.2 0)
 			(effects
@@
 			)
 		)
-		(property "PN" ""
+		(property "PN" "-"
 			(at 222.25 38.1 0)
 			(effects
@@
 			)
 		)
-		(property "MPN" ""
+		(property "MPN" "-"
 			(at 222.25 38.1 0)
 			(effects
@@
 			)
 		)
-		(property "MPN" ""
+		(property "MPN" "815-AISC-0603-R039-J"
 			(at 165.1 48.26 0)
 			(effects
@@
 			)
 		)
-		(property "PN" ""
+		(property "PN" "815-AISC-0603-R039-J"
 			(at 165.1 48.26 0)
 			(effects
@@
 			)
 		)
-		(property "PN" ""
+		(property "PN" "-"
 			(at 231.14 44.45 0)
 			(effects
@@
 			)
 		)
-		(property "MPN" ""
+		(property "MPN" "-"
 			(at 231.14 44.45 0)
 			(effects
@@
 			)
 		)
-		(property "PN" "C0603C104M5RAC7411"
+		(property "PN" "581-06035G104Z"
 			(at 102.87 139.7 0)
 			(effects
@@
 			)
 		)
-		(property "MPN" "C0603C104M5RAC7411"
+		(property "MPN" "581-06035G104Z"
 			(at 102.87 139.7 0)
 			(effects
@@
 			)
 		)
-		(property "PN" "C0603C104M5RAC7411"
+		(property "PN" "581-06035G104Z"
 			(at 96.52 107.95 0)
 			(effects
@@
 			)
 		)
-		(property "MPN" "C0603C104M5RAC7411"
+		(property "MPN" "581-06035G104Z"
 			(at 96.52 107.95 0)
 			(effects
@@
 			)
 		)
-		(property "PN" "C0603C104M5RAC7411"
+		(property "PN" "581-06035G104Z"
 			(at 93.98 139.7 0)
 			(effects
@@
 			)
 		)
-		(property "MPN" "C0603C104M5RAC7411"
+		(property "MPN" "581-06035G104Z"
 			(at 93.98 139.7 0)
 			(effects
@@
 			)
 		)
-		(property "PN" ""
+		(property "PN" "603-AC0603JRNP9BN270"
 			(at 143.51 48.26 0)
 			(effects
@@
 			)
 		)
-		(property "MPN" ""
+		(property "MPN" "603-AC0603JRNP9BN270"
 			(at 143.51 48.26 0)
 			(effects
@@
 			)
 		)
-		(property "PN" ""
+		(property "PN" "77-VJ0603A330KXAPBC"
 			(at 135.89 58.42 0)
 			(effects
@@
 			)
 		)
-		(property "MPN" ""
+		(property "MPN" "77-VJ0603A330KXAPBC"
 			(at 135.89 58.42 0)
 			(effects
@@
 			)
 		)
-		(property "PN" "C0603C103K5RAC7081"
+		(property "PN" "80-C0603C103M4RECLR"
 			(at 71.12 64.77 0)
 			(effects
@@
 			)
 		)
-		(property "MPN" "C0603C103K5RAC7081"
+		(property "MPN" "80-C0603C103M4RECLR"
 			(at 71.12 64.77 0)
 			(effects
@@
 			)
 		)
-		(property "PN" ""
+		(property "PN" "-"
 			(at 222.25 44.45 0)
 			(effects
@@
 			)
 		)
-		(property "MPN" ""
+		(property "MPN" "-"
 			(at 222.25 44.45 0)
 			(effects
@@
 			)
 		)
-		(property "PN" ""
+		(property "PN" "-"
 			(at 275.59 173.99 0)
 			(effects
@@
 			)
 		)
-		(property "MPN" ""
+		(property "MPN" "-"
 			(at 275.59 173.99 0)
 			(effects
@@
 			)
 		)
-		(property "PN" "C0603C103K5RAC7081"
+		(property "PN" "80-C0603C103M4RECLR"
 			(at 76.2 139.7 0)
 			(effects
@@
 			)
 		)
-		(property "MPN" "C0603C103K5RAC7081"
+		(property "MPN" "80-C0603C103M4RECLR"
 			(at 76.2 139.7 0)
 			(effects
@@
 			)
 		)
-		(property "PN" "C0603C104M5RAC7411"
+		(property "PN" "581-06035G104Z"
 			(at 85.09 139.7 0)
 			(effects
@@
 			)
 		)
-		(property "MPN" "C0603C104M5RAC7411"
+		(property "MPN" "581-06035G104Z"
 			(at 85.09 139.7 0)
 			(effects
@@
 			)
 		)
-		(property "PN" ""
+		(property "PN" "-"
 			(at 224.79 91.44 0)
 			(effects
@@
 			)
 		)
-		(property "MPN" ""
+		(property "MPN" "-"
 			(at 224.79 91.44 0)
 			(effects
@@
 			)
 		)
-		(property "PN" ""
+		(property "PN" "-"
 			(at 231.14 38.1 0)
 			(effects
@@
 			)
 		)
-		(property "MPN" ""
+		(property "MPN" "-"
 			(at 231.14 38.1 0)
 			(effects
@@
 			)
 		)
-		(property "PN" "C0603C104M5RAC7411"
+		(property "PN" "581-06035G104Z"
 			(at 105.41 107.95 0)
 			(effects
@@
 			)
 		)
-		(property "MPN" "C0603C104M5RAC7411"
+		(property "MPN" "581-06035G104Z"
 			(at 105.41 107.95 0)
 			(effects
@@
 			)
 		)
-		(property "MPN" ""
+		(property "MPN" "815-AISC-0603-R082-J"
 			(at 160.02 53.34 0)
 			(effects
@@
 			)
 		)
-		(property "PN" ""
+		(property "PN" "815-AISC-0603-R082-J"
 			(at 160.02 53.34 0)
 			(effects
@@
 			)
 		)
-		(property "PN" "C0603C103K5RAC7081"
+		(property "PN" "80-C0603C103M4RECLR"
 			(at 67.31 139.7 0)
 			(effects
@@
 			)
 		)
-		(property "MPN" "C0603C103K5RAC7081"
+		(property "MPN" "80-C0603C103M4RECLR"
 			(at 67.31 139.7 0)
 			(effects

Commit message: MPN fixes for Mouser
Parts:
- C1, C2, C3, C4: MPN 80-C0603C103M4RECLR -> C0603C103M4REC7411
- C10, C13, C5, C6, C7, C8, C9: MPN 581-06035G104Z -> 06035G104ZAT2A
- C11: MPN 77-VJ0603A330KXAPBC -> VJ0603A330KXAPW1BC
- C12: MPN 603-AC0603JRNP9BN270 -> AC0603JRNPO9BN270
- IC1: MPN 947-SX1255IWLTRT -> SX1255IWLTRT
- J1, J2: MPN 737-RF204AT0050G -> RF2-04A-T-00-50-G
- L1: MPN 815-AISC-0603-R082-J -> AISC-0603-R082J-T
- L2: MPN 815-AISC-0603-R039-J -> AISC-0603-R039J-T
Changed lines of the file:
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@@
 	(title_block
 		(title "SX1255 RPi Zero Shield")
-		(date "8-02-2025")
+		(date "10-02-2025")
 		(rev "A")
 		(company "M17 Foundation")
@@
 			)
 		)
-		(property "MPN" "581-06035G104Z"
+		(property "MPN" "06035G104ZAT2A"
 			(at 114.3 107.95 0)
 			(effects
@@
 			)
 		)
-		(property "MPN" "80-C0603C103M4RECLR"
+		(property "MPN" "C0603C103M4REC7411"
 			(at 58.42 139.7 0)
 			(effects
@@
 			)
 		)
-		(property "MPN" "581-06035G104Z"
+		(property "MPN" "06035G104ZAT2A"
 			(at 170.18 76.2 0)
 			(effects
@@
 			)
 		)
-		(property "MPN" "815-AISC-0603-R039-J"
+		(property "MPN" "AISC-0603-R039J-T"
 			(at 165.1 48.26 0)
 			(effects
@@
 			)
 		)
-		(property "MPN" "581-06035G104Z"
+		(property "MPN" "06035G104ZAT2A"
 			(at 102.87 139.7 0)
 			(effects
@@
 			)
 		)
-		(property "MPN" "581-06035G104Z"
+		(property "MPN" "06035G104ZAT2A"
 			(at 96.52 107.95 0)
 			(effects
@@
 			)
 		)
-		(property "MPN" "581-06035G104Z"
+		(property "MPN" "06035G104ZAT2A"
 			(at 93.98 139.7 0)
 			(effects
@@
 			)
 		)
-		(property "MPN" "603-AC0603JRNP9BN270"
+		(property "MPN" "AC0603JRNPO9BN270"
 			(at 143.51 48.26 0)
 			(effects
@@
 			)
 		)
-		(property "MPN" "77-VJ0603A330KXAPBC"
+		(property "MPN" "VJ0603A330KXAPW1BC"
 			(at 135.89 58.42 0)
 			(effects
@@
 			)
 		)
-		(property "MPN" "80-C0603C103M4RECLR"
+		(property "MPN" "C0603C103M4REC7411"
 			(at 71.12 64.77 0)
 			(effects
@@
 			)
 		)
-		(property "MPN" "737-RF204AT0050G"
+		(property "MPN" "RF2-04A-T-00-50-G"
 			(at 179.07 48.26 0)
 			(effects
@@
 			)
 		)
-		(property "MPN" "80-C0603C103M4RECLR"
+		(property "MPN" "C0603C103M4REC7411"
 			(at 76.2 139.7 0)
 			(effects
@@
 			)
 		)
-		(property "MPN" "737-RF204AT0050G"
+		(property "MPN" "RF2-04A-T-00-50-G"
 			(at 120.65 58.42 0)
 			(effects
@@
 			)
 		)
-		(property "MPN" "581-06035G104Z"
+		(property "MPN" "06035G104ZAT2A"
 			(at 85.09 139.7 0)
 			(effects
@@
 			)
 		)
-		(property "MPN" "581-06035G104Z"
+		(property "MPN" "06035G104ZAT2A"
 			(at 105.41 107.95 0)
 			(effects
@@
 			)
 		)
-		(property "MPN" "815-AISC-0603-R082-J"
+		(property "MPN" "AISC-0603-R082J-T"
 			(at 160.02 53.34 0)
 			(effects
@@
 			)
 		)
-		(property "MPN" "80-C0603C103M4RECLR"
+		(property "MPN" "C0603C103M4REC7411"
 			(at 67.31 139.7 0)
 			(effects
@@
 			)
 		)
-		(property "MPN" "947-SX1255IWLTRT"
+		(property "MPN" "SX1255IWLTRT"
 			(at 162.56 876.2 0)
 			(effects
